File: Tema 1 - Introducción al diseño mecatrónico/Tarea_1_Modulo_NRF24L01/Tarea_1_Modulo_NRF24L01.kicad_sch (KiCad schematic)
At the start: 21 parts, among them J1 Bus_de_datos, U1 NRF24L01, Y1 16MHz

Commit message: PCB completado
Parts:
- renumbered C8 to C1, C9 to C2, C1 to C3, C2 to C4, C3 to C5, C4 to C6, C5 to C8, C6 to C9
Changed lines of the file:
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@@
 		(dnp no)
 		(fields_autoplaced yes)
-		(property "Reference" "#PWR07"
+		(property "Reference" "#PWR09"
 			(at 168.91 139.7 0)
 			(effects
@@
 			(project "Tarea_1_Modulo_NRF24L01"
 				(path "/9c14c52e-195c-4085-91ab-23b919bd24f5"
-					(reference "#PWR07")
+					(reference "#PWR09")
 					(unit 1)
 				)
@@
 		(dnp no)
 		(fields_autoplaced yes)
-		(property "Reference" "#PWR01"
+		(property "Reference" "#PWR07"
 			(at 149.86 66.04 0)
 			(effects
@@
 			(project ""
 				(path "/9c14c52e-195c-4085-91ab-23b919bd24f5"
-					(reference "#PWR01")
+					(reference "#PWR07")
 					(unit 1)
 				)
@@
 		(dnp no)
 		(fields_autoplaced yes)
-		(property "Reference" "#PWR013"
+		(property "Reference" "#PWR05"
 			(at 129.54 77.47 0)
 			(effects
@@
 			(project "Tarea_1_Modulo_NRF24L01"
 				(path "/9c14c52e-195c-4085-91ab-23b919bd24f5"
-					(reference "#PWR013")
+					(reference "#PWR05")
 					(unit 1)
 				)
@@
 		(dnp no)
 		(fields_autoplaced yes)
-		(property "Reference" "#PWR011"
+		(property "Reference" "#PWR012"
 			(at 203.2 111.76 0)
 			(effects
@@
 			(project "Tarea_1_Modulo_NRF24L01"
 				(path "/9c14c52e-195c-4085-91ab-23b919bd24f5"
-					(reference "#PWR011")
+					(reference "#PWR012")
 					(unit 1)
 				)
@@
 		(dnp no)
 		(fields_autoplaced yes)
-		(property "Reference" "C5"
+		(property "Reference" "C8"
 			(at 205.74 100.3235 0)
 			(effects
@@
 			(project "Tarea_1_Modulo_NRF24L01"
 				(path "/9c14c52e-195c-4085-91ab-23b919bd24f5"
-					(reference "C5")
+					(reference "C8")
 					(unit 1)
 				)
@@
 		(dnp no)
 		(fields_autoplaced yes)
-		(property "Reference" "C9"
+		(property "Reference" "C2"
 			(at 132.08 66.0462 0)
 			(effects
@@
 			(project "Tarea_1_Modulo_NRF24L01"
 				(path "/9c14c52e-195c-4085-91ab-23b919bd24f5"
-					(reference "C9")
+					(reference "C2")
 					(unit 1)
 				)
@@
 		(dnp no)
 		(fields_autoplaced yes)
-		(property "Reference" "#PWR03"
+		(property "Reference" "#PWR06"
 			(at 132.08 124.46 0)
 			(effects
@@
 			(project "Tarea_1_Modulo_NRF24L01"
 				(path "/9c14c52e-195c-4085-91ab-23b919bd24f5"
-					(reference "#PWR03")
+					(reference "#PWR06")
 					(unit 1)
 				)
@@
 		(dnp no)
 		(fields_autoplaced yes)
-		(property "Reference" "C3"
+		(property "Reference" "C5"
 			(at 186.69 128.2762 0)
 			(effects
@@
 			(project "Tarea_1_Modulo_NRF24L01"
 				(path "/9c14c52e-195c-4085-91ab-23b919bd24f5"
-					(reference "C3")
+					(reference "C5")
 					(unit 1)
 				)
@@
 		(dnp no)
 		(fields_autoplaced yes)
-		(property "Reference" "C2"
+		(property "Reference" "C4"
 			(at 171.45 128.2762 0)
 			(effects
@@
 			(project "Tarea_1_Modulo_NRF24L01"
 				(path "/9c14c52e-195c-4085-91ab-23b919bd24f5"
-					(reference "C2")
+					(reference "C4")
 					(unit 1)
 				)
@@
 		(dnp no)
 		(fields_autoplaced yes)
-		(property "Reference" "#PWR010"
+		(property "Reference" "#PWR011"
 			(at 199.39 71.12 0)
 			(effects
@@
 			(project "Tarea_1_Modulo_NRF24L01"
 				(path "/9c14c52e-195c-4085-91ab-23b919bd24f5"
-					(reference "#PWR010")
+					(reference "#PWR011")
 					(unit 1)
 				)
@@
 		(dnp no)
 		(fields_autoplaced yes)
-		(property "Reference" "#PWR012"
+		(property "Reference" "#PWR03"
 			(at 119.38 77.47 0)
 			(effects
@@
 			(project "Tarea_1_Modulo_NRF24L01"
 				(path "/9c14c52e-195c-4085-91ab-23b919bd24f5"
-					(reference "#PWR012")
+					(reference "#PWR03")
 					(unit 1)
 				)
@@
 		(dnp no)
 		(fields_autoplaced yes)
-		(property "Reference" "#PWR08"
+		(property "Reference" "#PWR010"
 			(at 184.15 139.7 0)
 			(effects
@@
 			(project "Tarea_1_Modulo_NRF24L01"
 				(path "/9c14c52e-195c-4085-91ab-23b919bd24f5"
-					(reference "#PWR08")
+					(reference "#PWR010")
 					(unit 1)
 				)
@@
 		(dnp no)
 		(fields_autoplaced yes)
-		(property "Reference" "C4"
+		(property "Reference" "C6"
 			(at 195.5863 88.9 90)
 			(effects
@@
 			(project "Tarea_1_Modulo_NRF24L01"
 				(path "/9c14c52e-195c-4085-91ab-23b919bd24f5"
-					(reference "C4")
+					(reference "C6")
 					(unit 1)
 				)
@@
 		(dnp no)
 		(fields_autoplaced yes)
-		(property "Reference" "#PWR06"
+		(property "Reference" "#PWR01"
 			(at 109.22 85.09 0)
 			(effects
@@
 			(project "Tarea_1_Modulo_NRF24L01"
 				(path "/9c14c52e-195c-4085-91ab-23b919bd24f5"
-					(reference "#PWR06")
+					(reference "#PWR01")
 					(unit 1)
 				)
@@
 		(dnp no)
 		(fields_autoplaced yes)
-		(property "Reference" "C6"
+		(property "Reference" "C9"
 			(at 212.09 80.0162 0)
 			(effects
@@
 			(project "Tarea_1_Modulo_NRF24L01"
 				(path "/9c14c52e-195c-4085-91ab-23b919bd24f5"
-					(reference "C6")
+					(reference "C9")
 					(unit 1)
 				)
@@
 		(dnp no)
 		(fields_autoplaced yes)
-		(property "Reference" "#PWR05"
+		(property "Reference" "#PWR02"
 			(at 109.22 105.41 0)
 			(effects
@@
 			(project "Tarea_1_Modulo_NRF24L01"
 				(path "/9c14c52e-195c-4085-91ab-23b919bd24f5"
-					(reference "#PWR05")
+					(reference "#PWR02")
 					(unit 1)
 				)
@@
 		(dnp no)
 		(fields_autoplaced yes)
-		(property "Reference" "#PWR09"
+		(property "Reference" "#PWR013"
 			(at 209.55 71.12 0)
 			(effects
@@
 			(project "Tarea_1_Modulo_NRF24L01"
 				(path "/9c14c52e-195c-4085-91ab-23b919bd24f5"
-					(reference "#PWR09")
+					(reference "#PWR013")
 					(unit 1)
 				)
@@
 		(dnp no)
 		(fields_autoplaced yes)
-		(property "Reference" "#PWR02"
+		(property "Reference" "#PWR08"
 			(at 151.13 124.46 0)
 			(effects
@@
 			(project ""
 				(path "/9c14c52e-195c-4085-91ab-23b919bd24f5"
-					(reference "#PWR02")
+					(reference "#PWR08")
 					(unit 1)
 				)
@@
 		(dnp no)
 		(fields_autoplaced yes)
-		(property "Reference" "C8"
+		(property "Reference" "C1"
 			(at 121.92 66.0462 0)
 			(effects
@@
 			(project "Tarea_1_Modulo_NRF24L01"
 				(path "/9c14c52e-195c-4085-91ab-23b919bd24f5"
-					(reference "C8")
+					(reference "C1")
 					(unit 1)
 				)
@@
 		(dnp no)
 		(fields_autoplaced yes)
-		(property "Reference" "C1"
+		(property "Reference" "C3"
 			(at 134.62 113.0362 0)
 			(effects
@@
 			(project ""
 				(path "/9c14c52e-195c-4085-91ab-23b919bd24f5"
-					(reference "C1")
-					(unit 1)
-				)
+					(reference "C3")
+					(unit 1)
+				)
