File: Tema 4 - De requisitos a diseño mecatrónico/Tarea_2_Aislador_USB/Tarea_2_Aislador_USB.kicad_pcb (KiCad board)
At the start: 2 copper layers, 64 x 24 mm, 24 parts, among them IC1 NUP2202W1T2G, IC2 ADUM5000ARWZ, IC3 ADUM3160BRWZ, IC4 NUP2202W1T2G, J1 87520-0010BLF, J2 USB-B-S-F-B-TH-R

Commit message: Actualización del aislador USB
Parts:
- added D1: Green, PCM_JLCPCB:D_0603, F.Cu at (111.2, 86.5)
- added R10: 100Ω, PCM_JLCPCB:R_0603, F.Cu at (115.2, 86.5)
Connections:
- J1 pad MH1: unconnected-(J1-PadMH1) -> GND_A
- J1 pad MH2: unconnected-(J1-PadMH2) -> GND_A
- J2 pad MH1: unconnected-(J2-PadMH1) -> GND_B
- J2 pad MH2: unconnected-(J2-PadMH2) -> GND_B
Routing:
- net +5V: track 58.7 -> 65.6 mm
- net GND_B: track 7.56 -> 1.12 mm
- net GND_A: track 12.5 -> 10.0 mm
- net Net-(D1-Pad2): track 0.00 -> 2.36 mm
Other:
- board text added: "Yunely Sánchez Ruiz Marzo 2025"
